Commit message: removed unused sensors

File: prius_description/urdf/prius.urdf (robot description, URDF)
Before this commit: robot prius, 29 links, 28 joints
Links:
- removed link back_camera_link
- removed link back_camera_link_optical
- removed link back_left_far_sonar_link
- removed link back_left_middle_sonar_link
- removed link back_right_far_sonar_link
- removed link back_right_middle_sonar_link
- removed link front_left_far_sonar_link
- removed link front_left_laser_link
- removed link front_left_middle_sonar_link
- removed link front_right_far_sonar_link
- removed link front_right_laser_link
- removed link front_right_middle_sonar_link
- removed link left_camera_link
- removed link left_camera_link_optical
- removed link right_camera_link
- removed link right_camera_link_optical
- link front_camera_link: mass 1 -> 0.5
- link front_camera_link_optical: mass 1 -> 0.1
Joints:
- removed joint back_camera_joint
- removed joint back_camera_optical_joint
- removed joint back_left_far_sonar_joint
- removed joint back_left_middle_sonar_joint
- removed joint back_right_far_sonar_joint
- removed joint back_right_middle_sonar_joint
- removed joint front_left_far_sonar_joint
- removed joint front_left_laser_joint
- removed joint front_left_middle_sonar_joint
- removed joint front_right_far_sonar_joint
- removed joint front_right_laser_joint
- removed joint front_right_middle_sonar_joint
- removed joint left_camera_joint
- removed joint left_camera_optical_joint
- removed joint right_camera_joint
- removed joint right_camera_optical_joint
